File: Tecknik/plate/starter-Plate.kicad_pcb (KiCad board)
At the start: 2 copper layers, 231.6 x 76.2 mm, 0 parts

Commit message: updated plate
Other:
- board size 231.6 x 76.2 mm -> 231.4 x 76.1 mm
Changed lines of the file:
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@@
-(kicad_pcb (version 20171130) (host pcbnew 5.1.6-c6e7f7d~87~ubuntu20.04.1)
+(kicad_pcb (version 20171130) (host pcbnew "(5.1.10)-1")
   (general
     (thickness 1.6)
@@
     (aux_axis_origin 0 0)
     (grid_origin 641.97992 295.43248)
-    (visible_elements FFFFFF7F)
+    (visible_elements 7FFFFFFF)
     (pcbplotparams
       (layerselection 0x010fc_ffffffff)
@@
       (drillshape 0)
       (scaleselection 1)
-      (outputdirectory "ssssssss"))
+      (outputdirectory "ortho_plate_gerber"))
   )
   (net 0 "")
@@
     (uvia_drill 0.1)
   )
-  (gr_line (start 241.56538 12.9737) (end 15.94538 12.9737) (layer Edge.Cuts) (width 0.2))
+  (gr_line (start 241.46538 13.0237) (end 16.04538 13.0237) (layer Edge.Cuts) (width 0.2))
   (gr_circle (center 166.85538 52.1987) (end 167.85538 52.1987) (layer Edge.Cuts) (width 0.2))
-  (gr_line (start 244.56538 86.1737) (end 244.56538 15.9737) (layer Edge.Cuts) (width 0.2))
-  (gr_arc (start 15.94538 15.9737) (end 15.94538 12.9737) (angle -90) (layer Edge.Cuts) (width 0.2))
-  (gr_arc (start 241.56538 86.1737) (end 241.56538 89.1737) (angle -90) (layer Edge.Cuts) (width 0.2))
+  (gr_line (start 244.46538 86.1237) (end 244.46538 16.0237) (layer Edge.Cuts) (width 0.2))
+  (gr_arc (start 16.04538 16.0237) (end 16.04538 13.0237) (angle -90) (layer Edge.Cuts) (width 0.2))
+  (gr_arc (start 241.46538 86.1237) (end 241.46538 89.1237) (angle -90) (layer Edge.Cuts) (width 0.2))
   (gr_circle (center 90.65538 52.1987) (end 91.65538 52.1987) (layer Edge.Cuts) (width 0.2))
-  (gr_arc (start 241.56538 15.9737) (end 244.56538 15.9737) (angle -90) (layer Edge.Cuts) (width 0.2))
-  (gr_line (start 15.94538 89.1737) (end 241.56538 89.1737) (layer Edge.Cuts) (width 0.2))
+  (gr_arc (start 241.46538 16.0237) (end 244.46538 16.0237) (angle -90) (layer Edge.Cuts) (width 0.2))
+  (gr_line (start 16.04538 89.1237) (end 241.46538 89.1237) (layer Edge.Cuts) (width 0.2))
   (gr_circle (center 52.55538 68.3987) (end 53.55538 68.3987) (layer Edge.Cuts) (width 0.2))
   (gr_circle (center 224.00538 68.3987) (end 225.00538 68.3987) (layer Edge.Cuts) (width 0.2))
-  (gr_arc (start 15.94538 86.1737) (end 12.94538 86.1737) (angle -90) (layer Edge.Cuts) (width 0.2))
+  (gr_arc (start 16.04538 86.1237) (end 13.04538 86.1237) (angle -90) (layer Edge.Cuts) (width 0.2))
   (gr_circle (center 224.00538 32.2987) (end 225.00538 32.2987) (layer Edge.Cuts) (width 0.2))
   (gr_circle (center 33.50538 32.2987) (end 34.50538 32.2987) (layer Edge.Cuts) (width 0.2))
-  (gr_line (start 12.94538 15.9737) (end 12.94538 86.1737) (layer Edge.Cuts) (width 0.2))
+  (gr_line (start 13.04538 16.0237) (end 13.04538 86.1237) (layer Edge.Cuts) (width 0.2))
   (zone (net 0) (net_name "") (layer F.Cu) (hatch edge 0.508)
     (connect_pads (clearance 0.508))
     (min_thickness 0.254)
-    (fill (arc_segments 32) (thermal_gap 0.508) (thermal_bridge_width 0.508))
+    (fill yes (arc_segments 32) (thermal_gap 0.508) (thermal_bridge_width 0.508))
     (polygon
       (pts
@@
     (connect_pads (clearance 0.508))
     (min_thickness 0.254)
-    (fill (arc_segments 32) (thermal_gap 0.508) (thermal_bridge_width 0.508))
+    (fill yes (arc_segments 32) (thermal_gap 0.508) (thermal_bridge_width 0.508))
     (polygon
       (pts
